File: HornPCB.kicad_pcb (KiCad board)
At the start: 2 copper layers, 57 x 63 mm, 14 parts, among them J1 Conn_01x02, J2 Conn_01x02, J3 Conn_01x02, J4 Conn_01x02, Q1 IRLML0030, Q2 IRLML0030

Commit message: trace fix
Routing:
- net /HORN_SIG: track 40.8 -> 39.7 mm
Changed lines of the file:
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@@
 	)
 	(segment
-		(start 123.5 103.75)
-		(end 124.25 103.75)
+		(start 115.25 88.75)
+		(end 115.25 86.5)
 		(width 0.2)
 		(layer "B.Cu")
@@
 	)
 	(segment
-		(start 115.25 86.5)
+		(start 123.5 103)
+		(end 123.5 97)
+		(width 0.2)
+		(layer "B.Cu")
+		(net 4)
+	)
+	(segment
+		(start 123.5 97)
 		(end 115.25 88.75)
 		(width 0.2)
@@
 	)
 	(segment
-		(start 124.25 103.75)
-		(end 128 107.5)
+		(start 128 107.5)
+		(end 123.5 103)
 		(width 0.2)
 		(layer "B.Cu")
-		(net 4)
-	)
-	(segment
-		(start 121 94.5)
-		(end 122.25 94.5)
-		(width 0.2)
-		(layer "B.Cu")
-		(net 4)
-	)
-	(segment
-		(start 115.25 88.75)
-		(end 121 94.5)
-		(width 0.2)
-		(layer "B.Cu")
-		(net 4)
-	)
-	(segment
-		(start 123.5 95.75)
-		(end 123.5 103.75)
-		(width 0.2)
-		(layer "B.Cu")
-		(net 4)
-	)
-	(segment
-		(start 122.25 94.5)
-		(end 123.5 95.75)
-		(width 0.2)
-		(layer "B.Cu")
